Commit message: robot now goes around the 5

File: urdf/reactive_robot.urdf (robot description, URDF)
Before this commit: robot reactive_robot, 5 links, 4 joints
Links:
- added link rear_caster, mass 0.1; collision sphere radius=0.05; visual sphere radius=0.05
Joints:
- added joint rear_caster_joint: type fixed, parent base_link, child rear_caster, origin xyz=-0.1 0 -0.05 rpy=0 0 0
